File: hardware/mkm/mkm.kicad_pcb (KiCad board)
At the start: 2 copper layers, 60 x 65 mm, 26 parts, among them J1 DIN-5_180degree, J2 DIN-5_180degree, J3 DIN-5_180degree, U1 40106, U2 H11L1

Commit message: Sending simulated MIDI packets via BLE to the app (all in debug mode)
Parts:
- added D2: LED, LED_THT:LED_D5.0mm_Clear, F.Cu at (127.0, 53.2)
- added R7: 1k, Resistor_THT:R_Axial_DIN0207_L6.3mm_D2.5mm_P7.62mm_Horizontal, F.Cu at (120.8, 53.2)
- added SW1: SW_Push, Button_Switch_THT:SW_PUSH_6mm, F.Cu at (127.5, 102.5)
- moved C2 1.52 mm to (134.2, 80.0)
- moved U1 1.52 mm to (126.9, 83.9)
Connections:
- A1 pad 1: unconnected-(A1-GPIO0-Pad1) -> Net-(A1-GPIO0)
- A1 pad 20: unconnected-(A1-GPIO15-Pad20) -> Net-(A1-GPIO15)
Routing:
- net Net-(A1-GPIO15): track 0.00 -> 34.8 mm
- net Net-(A1-GPIO0): track 0.00 -> 12.1 mm
- net Net-(FB3-Pad1): track 0.00 -> 4.35 mm
- net Net-(D2-A): track 0.00 -> 3.67 mm
- net /TX: track 13.5 -> 14.9 mm
- net Net-(R4-Pad2): track 3.66 -> 4.53 mm
- net Net-(R3-Pad2): track 21.7 -> 20.9 mm
- net /RX: track 46.1 -> 45.6 mm
